File: Hardware/CLAS_Combo_Breakout/CLAS_Combo_Breakout.kicad_sch (KiCad schematic)
At the start: 80 parts, among them J1 USB_C_Receptacle_USB2.0, J2 USB_C_Receptacle_USB2.0, J3 Conn_SMA, U1 USBLC6-2P6, U10 NT1191GEAE3S, U2 ZED-F9P, U3 NEO-D9C-00B, U4 USBLC6-2P6, U5 LMV331, U6 AP2112K-3.3, U7 DSS20200, U8 PD0922J5050S2HF, U9 F2933NBGP

Commit message: 配置仮完了
Parts:
- removed D5: POWER, LED_SMD:LED_0603_1608Metric, symbol Device:LED_Small
- removed RN2: 1k, Resistor_SMD:R_Array_Convex_4x0402, symbol Device:R_Pack04
- added J2: ZED, Connector_PinHeader_2.54mm:PinHeader_1x11_P2.54mm_Vertical, symbol Connector_Generic:Conn_01x11
- added J3: NEO, Connector_PinHeader_2.54mm:PinHeader_1x09_P2.54mm_Vertical, symbol Connector_Generic:Conn_01x09
- added R17, R18, R19: 1k, Resistor_SMD:R_0603_1608Metric, symbol Device:R_Small
- renumbered D11 to D10, D4 to D3, D3 to D4, D6 to D5, D7 to D6, D8 to D7, D9 to D8, D10 to D9, J2 to J4, J3 to J5, R17 to R20, R18 to R21, R19 to R22, R20 to R23, R21 to R24, R22 to R25, R23 to R26, R24 to R27, R25 to R28, R26 to R29, R27 to R30
Connections:
- net +3.3V: now also J2.9 (Pin_9), J3.7 (Pin_7), R17.1
- net EXTANT_DETECT: now also J3.1 (Pin_1)
- net EXTINT_NEO: now also J3.3 (Pin_3)
- net EXTINT_ZED: now also J2.4 (Pin_4)
- net GEO: now also J2.2 (Pin_2), R18.1
- net GND: now also J2.8 (Pin_8), J3.6 (Pin_6)
- net RESET: now also J3.2 (Pin_2)
- net RTK: now also J2.3 (Pin_3)
- net RXD1_NEO: now also J3.4 (Pin_4)
- net RXD1_ZED: now also J2.6 (Pin_6)
- net SCL: now also J2.11 (Pin_11), J3.9 (Pin_9)
- net SDA: now also J2.10 (Pin_10), J3.8 (Pin_8)
- net TP: now also J2.1 (Pin_1), R19.1
- net TXD1_NEO: now also J3.5 (Pin_5)
- net TXD1_ZED: now also J2.7 (Pin_7)
- net TX_RDY: now also J2.5 (Pin_5)
- net at D6.2 (A): now also R19.2
- net at D5.2 (A): now also R18.2
- net at D4.2 (A): now also R17.2
Other:
- note removed: "3.3V LED"
- moved on the sheet: D4

Commit message: 配置完了
Parts:
- removed RN1: 33, Resistor_SMD:R_Array_Convex_4x0402, symbol Device:R_Pack04
- added R1, R3, R4, R6: 33, Resistor_SMD:R_0603_1608Metric, symbol Device:R_Small
- renumbered R6 to R10, R7 to R11, R8 to R12, R9 to R13, R10 to R14, R11 to R15, R12 to R16, R13 to R17, R14 to R18, R15 to R19, R1 to R2, R16 to R20, R17 to R21, R18 to R22, R19 to R23, R20 to R24, R21 to R25, R22 to R26, R23 to R27, R24 to R28, R25 to R29, R26 to R30, R27 to R31, R28 to R32, R29 to R33, R30 to R34, R2 to R5, R3 to R7, R4 to R8, R5 to R9
Connections:
- net RXD1_ZED: now also J2.5 (Pin_5); no longer J2.6 (Pin_6)
- net SCL: now also R3.2
- net SCL_ZED_: now also R3.1
- net SDA: now also R4.2
- net SDA_ZED_: now also R4.1
- net TXD1_ZED: now also J2.6 (Pin_6), R6.2; no longer J2.7 (Pin_7)
- net TXD1_ZED_: now also R6.1
- net TX_RDY: now also J2.7 (Pin_7), R1.2; no longer J2.5 (Pin_5)
- net TX_RDY_: now also R1.1

Commit message: 配線中
Connections:
- net EXTINT_NEO: now also J3.5 (Pin_5); no longer J3.3 (Pin_3)
- net RXD1_NEO: now also J3.3 (Pin_3); no longer J3.4 (Pin_4)
- net TXD1_NEO: now also J3.4 (Pin_4); no longer J3.5 (Pin_5)
Changed lines of the file:
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@@
     (effects (font (size 1.27 1.27)) (justify left bottom))
   )
-  (label "TXD1_NEO" (at 199.39 77.47 0)
+  (label "TXD1_NEO" (at 199.39 74.93 0)
     (effects (font (size 1.27 1.27)) (justify left bottom))
   )
@@
     (effects (font (size 1.27 1.27)) (justify left bottom))
   )
-  (label "RXD1_NEO" (at 199.39 74.93 0)
+  (label "RXD1_NEO" (at 199.39 72.39 0)
     (effects (font (size 1.27 1.27)) (justify left bottom))
   )
@@
     (effects (font (size 1.27 1.27)) (justify left bottom))
   )
-  (label "EXTINT_NEO" (at 199.39 72.39 0)
+  (label "EXTINT_NEO" (at 199.39 77.47 0)
     (effects (font (size 1.27 1.27)) (justify left bottom))
   )

Commit message: LED周りの配線を調整
Connections:
- net GEO: now also J2.1 (Pin_1); no longer J2.2 (Pin_2)
- net RTK: now also J2.2 (Pin_2); no longer J2.3 (Pin_3)
- net TP: now also J2.3 (Pin_3); no longer J2.1 (Pin_1)
Changed lines of the file:
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@@
     (effects (font (size 1.27 1.27)) (justify left bottom))
   )
-  (label "GEO" (at 177.8 64.77 180)
+  (label "GEO" (at 177.8 62.23 180)
     (effects (font (size 1.27 1.27)) (justify right bottom))
   )
-  (label "RTK" (at 177.8 67.31 180)
+  (label "RTK" (at 177.8 64.77 180)
     (effects (font (size 1.27 1.27)) (justify right bottom))
   )
@@
     (effects (font (size 1.27 1.27)) (justify right bottom))
   )
-  (label "TP" (at 177.8 62.23 180)
+  (label "TP" (at 177.8 67.31 180)
     (effects (font (size 1.27 1.27)) (justify right bottom))
   )
