File: Hardware/CLAS_Combo_Breakout_MovingBase-HAT/CLAS_Combo_Breakout_MovingBase-HAT.kicad_sch (KiCad schematic)
At the start: 64 parts, among them J1 MMCX, J2 SMA, J3 SWD, J4 ZED, J5 BATT, J6 NEO, J7 USB_C_Receptacle_USB2.0, Q1 AO3415A, SW1 SW_Push, SW2 SW_SPDT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

Commit message: 一部ライブラリを整理
Parts:
- added J8: RS485, Connector_JST:JST_PH_S3B-PH-K_1x03_P2.00mm_Horizontal, symbol Connector_Generic:Conn_01x03
- J5: footprint Connector_JST:JST_PH_S2B-PH-SM4-TB_1x02-1MP_P2.00mm_Horizontal -> Connector_JST:JST_PH_S2B-PH-K_1x02_P2.00mm_Horizontal
- U2: renamed from U?; footprint (none) -> Package_DFN_QFN_extlib:Texas_RMG0012A_1.8x1.8mm_P0.4mm
- U7: renamed from U?; footprint (none) -> Package_SO:SOIC-8_3.9x4.9mm_P1.27mm
- gave numbers to parts that had none: 6
Connections:
- net GND: now also J8.1 (Pin_1)
- net RS485_A: now also J8.3 (Pin_3)
- net RS485_B: now also J8.2 (Pin_2)
- net SWO: now reaches U3.41 (P0_18/TRCDAT0)
- net SWO: now also J3.6 (SWO/TDO)
- no-connect marks 12 -> 10
